File: PCB/CombinedLR/PhobGCC.kicad_sch (KiCad schematic)
At the start: 79 parts, among them J1 Conn_01x06_Female, J2 Conn_01x04_Female, J3 Conn_01x01_Male, J4 Conn_01x04_Male, J5 Conn_01x02_Male, J6 Button_Out, J7 Conn_01x02_Male, J8 Conn_01x02_Male, Q1 Q_NMOS_GSD, Q2 Q_PMOS_GDS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

Commit message: new mousebites and buttons
Parts:
- removed D1: D_Schottky_Shorted, wavbrd:D_SOD-523_Shorted, symbol Gamecube MB:D_Schottky_Shorted
- removed H21: MouseBiteLB, PhobGCC_Footprints:breakaway-mousebites, symbol Mechanical:MountingHole
- removed H23: MouseBiteRB, PhobGCC_Footprints:breakaway-mousebites, symbol Mechanical:MountingHole
- added F2: Fuse, wavbrd:R_1206_3216Metric, symbol Device:Fuse
- H14, H15: footprint wavbrd:mouse-bite-2.54mm-slot -> wavbrd:breakaway-mousebites-double
- H20: value MouseBiteLA -> MouseBiteL; footprint PhobGCC_Footprints:breakaway-mousebites -> wavbrd:breakaway-mousebites-double
- H21: renamed from H22; value MouseBiteRA -> MouseBiteR; footprint PhobGCC_Footprints:breakaway-mousebites -> wavbrd:breakaway-mousebites-double
- J7, J8: footprint Connector_PinHeader_2.54mm:PinHeader_1x02_P2.54mm_Vertical -> (none)
Connections:
- net Data: now also F2.2
- net at U1.9 (7_RX2_OUT1A): now also F2.1
Changed lines of the file:
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@@
       (effects (font (size 1 1)))
     )
-    (property "Footprint" "Connector_PinHeader_2.54mm:PinHeader_1x02_P2.54mm_Vertical" (id 2) (at 244.602 74.676 0)
+    (property "Footprint" "" (id 2) (at 244.602 74.676 0)
       (effects (font (size 1.27 1.27)) hide)
     )
@@
   (symbol (lib_id "Mechanical:MountingHole") (at 232.156 58.547 0) (unit 1)
     (in_bom yes) (on_board yes) (fields_autoplaced)
-    (property "Reference" "H22" (id 0) (at 234.696 57.7123 0)
-      (effects (font (size 1.27 1.27)) (justify left))
-    )
-    (property "Value" "MouseBiteRA" (id 1) (at 234.696 60.2492 0)
-      (effects (font (size 1.27 1.27)) (justify left))
-    )
-    (property "Footprint" "PhobGCC_Footprints:breakaway-mousebites" (id 2) (at 232.156 58.547 0)
+    (property "Reference" "H21" (id 0) (at 234.696 57.7123 0)
+      (effects (font (size 1.27 1.27)) (justify left))
+    )
+    (property "Value" "MouseBiteR" (id 1) (at 234.696 60.2492 0)
+      (effects (font (size 1.27 1.27)) (justify left))
+    )
+    (property "Footprint" "wavbrd:breakaway-mousebites-double" (id 2) (at 232.156 58.547 0)
       (effects (font (size 1.27 1.27)) hide)
     )
@@
       (effects (font (size 1.27 1.27)) (justify left))
     )
-    (property "Value" "MouseBiteLA" (id 1) (at 234.696 49.2002 0)
-      (effects (font (size 1.27 1.27)) (justify left))
-    )
-    (property "Footprint" "PhobGCC_Footprints:breakaway-mousebites" (id 2) (at 232.156 47.498 0)
+    (property "Value" "MouseBiteL" (id 1) (at 234.696 49.2002 0)
+      (effects (font (size 1.27 1.27)) (justify left))
+    )
+    (property "Footprint" "wavbrd:breakaway-mousebites-double" (id 2) (at 232.156 47.498 0)
       (effects (font (size 1.27 1.27)) hide)
     )
     (property "Datasheet" "~" (id 3) (at 232.156 47.498 0)
-      (effects (font (size 1.27 1.27)) hide)
-    )
-  )
-  (symbol (lib_id "Mechanical:MountingHole") (at 232.156 64.262 0) (unit 1)
-    (in_bom yes) (on_board yes) (fields_autoplaced)
-    (property "Reference" "H23" (id 0) (at 234.696 63.4273 0)
-      (effects (font (size 1.27 1.27)) (justify left))
-    )
-    (property "Value" "MouseBiteRB" (id 1) (at 234.696 65.9642 0)
-      (effects (font (size 1.27 1.27)) (justify left))
-    )
-    (property "Footprint" "PhobGCC_Footprints:breakaway-mousebites" (id 2) (at 232.156 64.262 0)
-      (effects (font (size 1.27 1.27)) hide)
-    )
-    (property "Datasheet" "~" (id 3) (at 232.156 64.262 0)
       (effects (font (size 1.27 1.27)) hide)
     )
@@
       (effects (font (size 1.27 1.27)) (justify left))
     )
-    (property "Footprint" "wavbrd:mouse-bite-2.54mm-slot" (id 2) (at 200.66 128.651 0)
+    (property "Footprint" "wavbrd:breakaway-mousebites-double" (id 2) (at 200.66 128.651 0)
       (effects (font (size 1.27 1.27)) hide)
     )
@@
       (effects (font (size 1 1)))
     )
-    (property "Footprint" "Connector_PinHeader_2.54mm:PinHeader_1x02_P2.54mm_Vertical" (id 2) (at 244.602 84.074 0)
+    (property "Footprint" "" (id 2) (at 244.602 84.074 0)
       (effects (font (size 1.27 1.27)) hide)
     )
@@
     (pin "2")
     (pin "3")
-  )
-  (symbol (lib_id "Mechanical:MountingHole") (at 232.156 53.213 0) (unit 1)
-    (in_bom yes) (on_board yes) (fields_autoplaced)
-    (property "Reference" "H21" (id 0) (at 234.696 52.3783 0)
-      (effects (font (size 1.27 1.27)) (justify left))
-    )
-    (property "Value" "MouseBiteLB" (id 1) (at 234.696 54.9152 0)
-      (effects (font (size 1.27 1.27)) (justify left))
-    )
-    (property "Footprint" "PhobGCC_Footprints:breakaway-mousebites" (id 2) (at 232.156 53.213 0)
-      (effects (font (size 1.27 1.27)) hide)
-    )
-    (property "Datasheet" "~" (id 3) (at 232.156 53.213 0)
-      (effects (font (size 1.27 1.27)) hide)
-    )
   )
   (symbol (lib_id "Device:Q_PMOS_GSD") (at 90.17 27.94 0) (mirror x) (unit 1)
@@
     (pin "2")
   )
-  (symbol (lib_id "Gamecube MB:D_Schottky_Shorted") (at 33.02 96.52 90) (unit 1)
-    (in_bom yes) (on_board yes)
-    (property "Reference" "D1" (id 0) (at 26.67 95.25 90)
-      (effects (font (size 1.27 1.27)) (justify right))
-    )
-    (property "Value" "D_Schottky_Shorted" (id 1) (at 21.59 101.6 90)
-      (effects (font (size 1.27 1.27)) (justify right))
-    )
-    (property "Footprint" "wavbrd:D_SOD-523_Shorted" (id 2) (at 33.02 96.52 0)
-      (effects (font (size 1.27 1.27)) hide)
-    )
-    (property "Datasheet" "~" (id 3) (at 33.02 96.52 0)
-      (effects (font (size 1.27 1.27)) hide)
-    )
-    (pin "1")
-    (pin "2")
-  )
   (symbol (lib_id "power:GND") (at 249.809 36.703 0) (unit 1)
     (in_bom yes) (on_board yes) (fields_autoplaced)
@@
       (effects (font (size 1.27 1.27)) (justify left))
     )
-    (property "Footprint" "wavbrd:mouse-bite-2.54mm-slot" (id 2) (at 200.66 134.366 0)
+    (property "Footprint" "wavbrd:breakaway-mousebites-double" (id 2) (at 200.66 134.366 0)
       (effects (font (size 1.27 1.27)) hide)
     )
@@
       (effects (font (size 1.27 1.27)) hide)
     )
+  )
+  (symbol (lib_id "Device:Fuse") (at 33.02 96.52 0) (unit 1)
+    (in_bom yes) (on_board yes) (fields_autoplaced)
+    (property "Reference" "F2" (id 0) (at 34.544 95.6115 0)
+      (effects (font (size 1.27 1.27)) (justify left))
+    )
+    (property "Value" "Fuse" (id 1) (at 34.544 98.3866 0)
+      (effects (font (size 1.27 1.27)) (justify left))
+    )
+    (property "Footprint" "wavbrd:R_1206_3216Metric" (id 2) (at 31.242 96.52 90)
+      (effects (font (size 1.27 1.27)) hide)
+    )
+    (property "Datasheet" "~" (id 3) (at 33.02 96.52 0)
+      (effects (font (size 1.27 1.27)) hide)
+    )
+    (property "LCSC" "C69680" (id 4) (at 33.02 96.52 0)
+      (effects (font (size 1.27 1.27)) hide)
+    )
+    (property "MPN" "" (id 5) (at 33.02 96.52 0)
+      (effects (font (size 1.27 1.27)) hide)
+    )
+    (property "Manufacturer" "" (id 6) (at 33.02 96.52 0)
+      (effects (font (size 1.27 1.27)) hide)
+    )
+    (pin "1")
+    (pin "2")
   )
   (symbol (lib_id "power:GND") (at 120.65 66.04 0) (unit 1)
@@
       (reference "C13") (unit 1) (value "1u") (footprint "wavbrd:C_0603_1608Metric_Pad1.08x0.95mm_HandSolder")
     )
-    (path "/dc7d42fa-0e8f-4624-9dce-327f10f7c7de"
-      (reference "D1") (unit 1) (value "D_Schottky_Shorted") (footprint "wavbrd:D_SOD-523_Shorted")
-    )
     (path "/214e41d3-ead9-4e70-8205-61f67874e54d"
       (reference "D2") (unit 1) (value "M7C") (footprint "wavbrd:D_SOD-123")
@@
       (reference "F1") (unit 1) (value "Fuse") (footprint "wavbrd:R_1206_3216Metric")
     )
+    (path "/fb653c74-ba25-4919-b551-a8fd09bbe12d"
+      (reference "F2") (unit 1) (value "Fuse") (footprint "wavbrd:R_1206_3216Metric")
+    )
     (path "/00000000-0000-0000-0000-000061ce47a0"
       (reference "H1") (unit 1) (value "5.2mm") (footprint "wavbrd:MountingHole_5.2mm")
@@
     )
     (path "/c47d0840-d558-41d0-b705-7adf6c7e6a54"
-      (reference "H14") (unit 1) (value "MouseBite") (footprint "wavbrd:mouse-bite-2.54mm-slot")
+      (reference "H14") (unit 1) (value "MouseBite") (footprint "wavbrd:breakaway-mousebites-double")
     )
     (path "/f929878e-6040-433f-956c-7a368fa106d8"
-      (reference "H15") (unit 1) (value "MouseBite") (footprint "wavbrd:mouse-bite-2.54mm-slot")
+      (reference "H15") (unit 1) (value "MouseBite") (footprint "wavbrd:breakaway-mousebites-double")
     )
     (path "/6b393128-7714-47bd-9d6f-caa4e2bd427c"
@@
     )
     (path "/9caa825e-43a9-45d3-8dad-ce1e46623c13"
-      (reference "H20") (unit 1) (value "MouseBiteLA") (footprint "PhobGCC_Footprints:breakaway-mousebites")
-    )
-    (path "/d3e7f16d-a250-4de7-87e5-9bc710a55c24"
-      (reference "H21") (unit 1) (value "MouseBiteLB") (footprint "PhobGCC_Footprints:breakaway-mousebites")
+      (reference "H20") (unit 1) (value "MouseBiteL") (footprint "wavbrd:breakaway-mousebites-double")
     )
     (path "/47f8e668-273a-44f0-a487-9421f049d27f"
-      (reference "H22") (unit 1) (value "MouseBiteRA") (footprint "PhobGCC_Footprints:breakaway-mousebites")
-    )
-    (path "/9ffa7a41-84e2-439f-ab9e-a1334179edc6"
-      (reference "H23") (unit 1) (value "MouseBiteRB") (footprint "PhobGCC_Footprints:breakaway-mousebites")
+      (reference "H21") (unit 1) (value "MouseBiteR") (footprint "wavbrd:breakaway-mousebites-double")
     )
     (path "/00000000-0000-0000-0000-000061572882"
@@
     )
     (path "/0206e765-825a-4e51-9371-9f239143e77c"
-      (reference "J7") (unit 1) (value "Conn_01x02_Male") (footprint "Connector_PinHeader_2.54mm:PinHeader_1x02_P2.54mm_Vertical")
+      (reference "J7") (unit 1) (value "Conn_01x02_Male") (footprint "wavbrd:PinHeader_1x02_P2.54mm_Vertical")
     )
     (path "/c970f863-2eeb-4363-945c-2275a112fd4c"
-      (reference "J8") (unit 1) (value "Conn_01x02_Male") (footprint "Connector_PinHeader_2.54mm:PinHeader_1x02_P2.54mm_Vertical")
+      (reference "J8") (unit 1) (value "Conn_01x02_Male") (footprint "wavbrd:PinHeader_1x02_P2.54mm_Vertical")
     )
     (path "/d2da7f57-ee9e-4fd2-ab66-6ced21a875ef"

Commit message: 1.2.2 update
Parts:
- removed F2: Fuse, wavbrd:R_1206_3216Metric, symbol Device:Fuse
- added D1: D_Schottky_Shorted, wavbrd:D_SOD-523_Shorted, symbol PhobGCC_Symbol_Library:D_Schottky_Shorted
- D3: footprint wavbrd:D_SOD-123 -> (none)
- J7, J8: footprint (none) -> wavbrd:PinHeader_1x02_P2.54mm_Vertical
Connections:
- net Data: now also U1.9 (7_RX2_OUT1A), D1.1 (K), D1.2 (A)
Changed lines of the file:
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@@
   (junction (at 120.65 63.5) (diameter 0) (color 0 0 0 0)
   )
+  (junction (at 185.039 32.258) (diameter 0) (color 0 0 0 0)
+  )
+  (junction (at 62.23 38.1) (diameter 0) (color 0 0 0 0)
+  )
+  (junction (at 177.8 34.29) (diameter 0) (color 0 0 0 0)
+  )
+  (junction (at 76.2 168.91) (diameter 0) (color 0 0 0 0)
+  )
+  (junction (at 99.06 180.34) (diameter 0) (color 0 0 0 0)
+  )
+  (junction (at 249.809 32.258) (diameter 0) (color 0 0 0 0)
+  )
+  (junction (at 177.8 86.36) (diameter 0) (color 0 0 0 0)
+  )
+  (junction (at 33.02 92.71) (diameter 0) (color 0 0 0 0)
+  )
+  (junction (at 177.8 120.65) (diameter 0) (color 0 0 0 0)
+  )
+  (junction (at 114.3 180.34) (diameter 0) (color 0 0 0 0)
+  )
+  (junction (at 99.06 54.61) (diameter 0) (color 0 0 0 0)
+  )
+  (junction (at 40.64 180.34) (diameter 0) (color 0 0 0 0)
+  )
+  (junction (at 177.8 74.93) (diameter 0) (color 0 0 0 0)
+  )
+  (junction (at 26.67 39.37) (diameter 0) (color 0 0 0 0)
+  )
+  (junction (at 118.11 123.19) (diameter 0) (color 0 0 0 0)
+  )
   (junction (at 109.22 113.03) (diameter 0) (color 0 0 0 0)
   )
-  (junction (at 185.039 32.258) (diameter 0) (color 0 0 0 0)
-  )
-  (junction (at 62.23 38.1) (diameter 0) (color 0 0 0 0)
-  )
-  (junction (at 177.8 34.29) (diameter 0) (color 0 0 0 0)
-  )
-  (junction (at 76.2 168.91) (diameter 0) (color 0 0 0 0)
-  )
-  (junction (at 99.06 180.34) (diameter 0) (color 0 0 0 0)
-  )
-  (junction (at 249.809 32.258) (diameter 0) (color 0 0 0 0)
-  )
-  (junction (at 177.8 86.36) (diameter 0) (color 0 0 0 0)
-  )
-  (junction (at 177.8 120.65) (diameter 0) (color 0 0 0 0)
-  )
-  (junction (at 114.3 180.34) (diameter 0) (color 0 0 0 0)
-  )
-  (junction (at 99.06 54.61) (diameter 0) (color 0 0 0 0)
-  )
-  (junction (at 40.64 180.34) (diameter 0) (color 0 0 0 0)
-  )
-  (junction (at 177.8 74.93) (diameter 0) (color 0 0 0 0)
-  )
-  (junction (at 26.67 39.37) (diameter 0) (color 0 0 0 0)
-  )
-  (junction (at 118.11 123.19) (diameter 0) (color 0 0 0 0)
-  )
   (junction (at 80.01 27.94) (diameter 0) (color 0 0 0 0)
   )
@@
   )
   (junction (at 76.2 180.34) (diameter 0) (color 0 0 0 0)
+  )
+  (junction (at 33.02 100.33) (diameter 0) (color 0 0 0 0)
   )
   (junction (at 40.64 168.91) (diameter 0) (color 0 0 0 0)
@@
     (stroke (width 0) (type default) (color 0 0 0 0))
   )
+  (wire (pts (xy 33.02 92.71) (xy 33.02 93.98))
+    (stroke (width 0) (type default) (color 0 0 0 0))
+  )
   (wire (pts (xy 156.21 95.25) (xy 177.8 95.25))
     (stroke (width 0) (type default) (color 0 0 0 0))
@@
     (stroke (width 0) (type default) (color 0 0 0 0))
   )
+  (wire (pts (xy 33.02 99.06) (xy 33.02 100.33))
+    (stroke (width 0) (type default) (color 0 0 0 0))
+  )
   (wire (pts (xy 52.07 168.91) (xy 43.18 168.91))
     (stroke (width 0) (type default) (color 0 0 0 0))
@@
     (stroke (width 0) (type default) (color 0 0 0 0))
   )
+  (wire (pts (xy 30.48 93.98) (xy 30.48 99.06))
+    (stroke (width 0) (type default) (color 0 0 0 0))
+  )
   (wire (pts (xy 111.76 125.73) (xy 114.3 125.73))
     (stroke (width 0) (type default) (color 0 0 0 0))
@@
     (stroke (width 0) (type default) (color 0 0 0 0))
   )
+  (wire (pts (xy 30.48 99.06) (xy 33.02 99.06))
+    (stroke (width 0) (type default) (color 0 0 0 0))
+  )
   (wire (pts (xy 242.57 148.59) (xy 251.46 148.59))
     (stroke (width 0) (type default) (color 0 0 0 0))
@@
   )
   (wire (pts (xy 118.11 123.19) (xy 129.54 123.19))
+    (stroke (width 0) (type default) (color 0 0 0 0))
+  )
+  (wire (pts (xy 33.02 93.98) (xy 30.48 93.98))
     (stroke (width 0) (type default) (color 0 0 0 0))
   )
@@
       (effects (font (size 1 1)))
     )
-    (property "Footprint" "" (id 2) (at 244.602 74.676 0)
+    (property "Footprint" "wavbrd:PinHeader_1x02_P2.54mm_Vertical" (id 2) (at 244.602 74.676 0)
       (effects (font (size 1.27 1.27)) hide)
     )
@@
     (pin "1")
   )
+  (symbol (lib_id "Device:D_Schottky") (at 109.22 109.22 90) (unit 1)
+    (in_bom yes) (on_board yes)
+    (property "Reference" "D3" (id 0) (at 104.14 109.22 0))
+    (property "Value" "M7C" (id 1) (at 106.68 109.22 0))
+    (property "Footprint" "" (id 2) (at 109.22 109.22 0)
+      (effects (font (size 1.27 1.27)) hide)
+    )
+    (property "Datasheet" "~" (id 3) (at 109.22 109.22 0)
+      (effects (font (size 1.27 1.27)) hide)
+    )
+    (property "JLCPN" "" (id 4) (at 109.22 109.22 0)
+      (effects (font (size 1.27 1.27)) hide)
+    )
+    (property "LCSC" "C8598" (id 5) (at 109.22 109.22 0)
+      (effects (font (size 1.27 1.27)) hide)
+    )
+    (property "MPN" "" (id 6) (at 109.22 109.22 0)
+      (effects (font (size 1.27 1.27)) hide)
+    )
+    (property "Manufacturer" "" (id 7) (at 109.22 109.22 0)
+      (effects (font (size 1.27 1.27)) hide)
+    )
+    (pin "1")
+    (pin "2")
+  )
   (symbol (lib_id "Mechanical:MountingHole") (at 200.66 140.208 0) (unit 1)
     (in_bom yes) (on_board yes) (fields_autoplaced)
@@
     )
     (property "Manufacturer" "" (id 6) (at 72.39 168.91 0)
+      (effects (font (size 1.27 1.27)) hide)
+    )
+    (pin "1")
+    (pin "2")
+  )
+  (symbol (lib_id "PhobGCC_Symbol_Library:D_Schottky_Shorted") (at 33.02 96.52 90) (unit 1)
+    (in_bom yes) (on_board yes) (fields_autoplaced)
+    (property "Reference" "D1" (id 0) (at 35.052 95.6853 90)
+      (effects (font (size 1.27 1.27)) (justify right))
+    )
+    (property "Value" "D_Schottky_Shorted" (id 1) (at 35.052 98.2222 90)
+      (effects (font (size 1.27 1.27)) (justify right))
+    )
+    (property "Footprint" "wavbrd:D_SOD-523_Shorted" (id 2) (at 33.02 96.52 0)
+      (effects (font (size 1.27 1.27)) hide)
+    )
+    (property "Datasheet" "~" (id 3) (at 33.02 96.52 0)
       (effects (font (size 1.27 1.27)) hide)
     )
@@
     (pin "9")
   )
-  (symbol (lib_id "Device:D_Schottky") (at 109.22 109.22 90) (unit 1)
-    (in_bom yes) (on_board yes)
-    (property "Reference" "D3" (id 0) (at 104.14 109.22 0))
-    (property "Value" "M7C" (id 1) (at 106.68 109.22 0))
-    (property "Footprint" "wavbrd:D_SOD-123" (id 2) (at 109.22 109.22 0)
-      (effects (font (size 1.27 1.27)) hide)
-    )
-    (property "Datasheet" "~" (id 3) (at 109.22 109.22 0)
-      (effects (font (size 1.27 1.27)) hide)
-    )
-    (property "JLCPN" "" (id 4) (at 109.22 109.22 0)
-      (effects (font (size 1.27 1.27)) hide)
-    )
-    (property "LCSC" "C8598" (id 5) (at 109.22 109.22 0)
-      (effects (font (size 1.27 1.27)) hide)
-    )
-    (property "MPN" "" (id 6) (at 109.22 109.22 0)
-      (effects (font (size 1.27 1.27)) hide)
-    )
-    (property "Manufacturer" "" (id 7) (at 109.22 109.22 0)
-      (effects (font (size 1.27 1.27)) hide)
-    )
-    (pin "1")
-    (pin "2")
-  )
   (symbol (lib_id "Mechanical:MountingHole") (at 200.66 128.651 0) (unit 1)
     (in_bom yes) (on_board yes) (fields_autoplaced)
@@
       (effects (font (size 1 1)))
     )
-    (property "Footprint" "" (id 2) (at 244.602 84.074 0)
+    (property "Footprint" "wavbrd:PinHeader_1x02_P2.54mm_Vertical" (id 2) (at 244.602 84.074 0)
       (effects (font (size 1.27 1.27)) hide)
     )
@@
     )
   )
-  (symbol (lib_id "Device:Fuse") (at 33.02 96.52 0) (unit 1)
-    (in_bom yes) (on_board yes) (fields_autoplaced)
-    (property "Reference" "F2" (id 0) (at 34.544 95.6115 0)
-      (effects (font (size 1.27 1.27)) (justify left))
-    )
-    (property "Value" "Fuse" (id 1) (at 34.544 98.3866 0)
-      (effects (font (size 1.27 1.27)) (justify left))
-    )
-    (property "Footprint" "wavbrd:R_1206_3216Metric" (id 2) (at 31.242 96.52 90)
-      (effects (font (size 1.27 1.27)) hide)
-    )
-    (property "Datasheet" "~" (id 3) (at 33.02 96.52 0)
-      (effects (font (size 1.27 1.27)) hide)
-    )
-    (property "LCSC" "C69680" (id 4) (at 33.02 96.52 0)
-      (effects (font (size 1.27 1.27)) hide)
-    )
-    (property "MPN" "" (id 5) (at 33.02 96.52 0)
-      (effects (font (size 1.27 1.27)) hide)
-    )
-    (property "Manufacturer" "" (id 6) (at 33.02 96.52 0)
-      (effects (font (size 1.27 1.27)) hide)
-    )
-    (pin "1")
-    (pin "2")
-  )
   (symbol (lib_id "power:GND") (at 120.65 66.04 0) (unit 1)
     (in_bom yes) (on_board yes)
@@
       (reference "C13") (unit 1) (value "1u") (footprint "wavbrd:C_0603_1608Metric_Pad1.08x0.95mm_HandSolder")
     )
+    (path "/bcd1d003-705a-4a74-aa1b-8b1527ce112a"
+      (reference "D1") (unit 1) (value "D_Schottky_Shorted") (footprint "wavbrd:D_SOD-523_Shorted")
+    )
     (path "/214e41d3-ead9-4e70-8205-61f67874e54d"
       (reference "D2") (unit 1) (value "M7C") (footprint "wavbrd:D_SOD-123")
     )
-    (path "/c45ca1ab-50a8-4158-9b8e-86eb478b26b1"
+    (path "/65840528-ae86-4ed9-af78-7b21e0f683c8"
       (reference "D3") (unit 1) (value "M7C") (footprint "wavbrd:D_SOD-123")
     )
@@
       (reference "F1") (unit 1) (value "Fuse") (footprint "wavbrd:R_1206_3216Metric")
     )
-    (path "/fb653c74-ba25-4919-b551-a8fd09bbe12d"
-      (reference "F2") (unit 1) (value "Fuse") (footprint "wavbrd:R_1206_3216Metric")
-    )
     (path "/00000000-0000-0000-0000-000061ce47a0"

Commit message: 1.2.3 update
Parts:
- D3: footprint (none) -> wavbrd:D_SOD-123
- J2: footprint wavbrd:Pin_Header_Straight_1x04_Pitch2.00mm -> wavbrd:PinHeader_1x04_P2.00mm_Vertical
- SW8: footprint wavbrd:Z_Switch_Edge -> (none)
Changed lines of the file:
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@@
       (effects (font (size 1.27 1.27)) (justify left))
     )
-    (property "Footprint" "wavbrd:Pin_Header_Straight_1x04_Pitch2.00mm" (id 2) (at 248.92 105.41 0)
+    (property "Footprint" "wavbrd:PinHeader_1x04_P2.00mm_Vertical" (id 2) (at 248.92 105.41 0)
       (effects (font (size 1.27 1.27)) hide)
     )
@@
     (property "Reference" "SW8" (id 0) (at 148.59 88.9 0))
     (property "Value" "1825027-5" (id 1) (at 148.59 91.44 0))
-    (property "Footprint" "wavbrd:Z_Switch_Edge" (id 2) (at 148.59 95.25 0)
+    (property "Footprint" "" (id 2) (at 148.59 95.25 0)
       (effects (font (size 1.27 1.27)) hide)
     )
@@
     (property "Reference" "D3" (id 0) (at 104.14 109.22 0))
     (property "Value" "M7C" (id 1) (at 106.68 109.22 0))
-    (property "Footprint" "" (id 2) (at 109.22 109.22 0)
+    (property "Footprint" "wavbrd:D_SOD-123" (id 2) (at 109.22 109.22 0)
       (effects (font (size 1.27 1.27)) hide)
     )
@@
     )
     (path "/00000000-0000-0000-0000-000061575d66"
-      (reference "J2") (unit 1) (value "Conn_01x04_Female") (footprint "wavbrd:Pin_Header_Straight_1x04_Pitch2.00mm")
+      (reference "J2") (unit 1) (value "Conn_01x04_Female") (footprint "wavbrd:PinHeader_1x04_P2.00mm_Vertical")
     )
     (path "/00000000-0000-0000-0000-000061cbc92e"
@@
     )
     (path "/00000000-0000-0000-0000-00006159dc5a"
-      (reference "SW8") (unit 1) (value "1825027-5") (footprint "wavbrd:Z_Switch_Edge")
+      (reference "SW8") (unit 1) (value "1825027-5") (footprint "wavbrd:Z_Switch_Edge_Omron")
     )
     (path "/00000000-0000-0000-0000-00006157aadd"
