File: PCB/CombinedLR/PhobGCC.kicad_sch (KiCad schematic)
At the start: 77 parts, among them J1 Conn_01x06_Female, J2 Conn_01x04_Female, J3 Conn_01x01_Male, J4 Conn_01x04_Male, J5 Conn_01x02_Male, J6 Button_Out, J7 Conn_01x02_Male, J8 Conn_01x02_Male, Q1 Q_NMOS_GSD, Q2 Q_PMOS_GDS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

Commit message: 1.2.X final tweaks
Parts:
- added J9: Conn_01x02_Male, symbol Connector:Conn_01x02_Male
- SW8: footprint (none) -> wavbrd:Z_Switch_Edge_Omron
Connections:
- net +5V: now also J9.1 (Pin_1)
- net at D2.2 (A), F1.1, J5.2 (Pin_2)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: now also J9.2 (Pin_2)
Changed lines of the file:
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@@
   (junction (at 249.809 36.703) (diameter 0) (color 0 0 0 0)
   )
+  (junction (at 120.65 28.956) (diameter 0) (color 0 0 0 0)
+  )
   (junction (at 120.65 22.86) (diameter 0) (color 0 0 0 0)
   )
@@
   (junction (at 120.65 33.02) (diameter 0) (color 0 0 0 0)
   )
+  (junction (at 120.65 24.384) (diameter 0) (color 0 0 0 0)
+  )
   (junction (at 185.039 55.118) (diameter 0) (color 0 0 0 0)
   )
@@
     (stroke (width 0) (type default) (color 0 0 0 0))
   )
+  (wire (pts (xy 127.508 24.384) (xy 120.65 24.384))
+    (stroke (width 0) (type default) (color 0 0 0 0))
+  )
   (wire (pts (xy 259.969 55.626) (xy 266.827 55.626))
     (stroke (width 0) (type default) (color 0 0 0 0))
@@
     (stroke (width 0) (type default) (color 0 0 0 0))
   )
-  (wire (pts (xy 120.65 27.94) (xy 120.65 33.02))
+  (wire (pts (xy 120.65 27.94) (xy 120.65 28.956))
     (stroke (width 0) (type default) (color 0 0 0 0))
   )
@@
     (stroke (width 0) (type default) (color 0 0 0 0))
   )
+  (wire (pts (xy 120.65 28.956) (xy 120.65 33.02))
+    (stroke (width 0) (type default) (color 0 0 0 0))
+  )
   (wire (pts (xy 185.039 32.258) (xy 185.039 24.638))
     (stroke (width 0) (type default) (color 0 0 0 0))
@@
     (stroke (width 0) (type default) (color 0 0 0 0))
   )
+  (wire (pts (xy 127.508 25.4) (xy 127.508 24.384))
+    (stroke (width 0) (type default) (color 0 0 0 0))
+  )
   (wire (pts (xy 163.83 34.29) (xy 154.94 34.29))
     (stroke (width 0) (type default) (color 0 0 0 0))
@@
     (stroke (width 0) (type default) (color 0 0 0 0))
   )
+  (wire (pts (xy 127.508 27.94) (xy 127.508 28.956))
+    (stroke (width 0) (type default) (color 0 0 0 0))
+  )
   (wire (pts (xy 173.99 143.51) (xy 177.8 143.51))
     (stroke (width 0) (type default) (color 0 0 0 0))
@@
     (stroke (width 0) (type default) (color 0 0 0 0))
   )
+  (wire (pts (xy 120.65 24.384) (xy 120.65 25.4))
+    (stroke (width 0) (type default) (color 0 0 0 0))
+  )
   (wire (pts (xy 48.26 138.43) (xy 41.91 138.43))
     (stroke (width 0) (type default) (color 0 0 0 0))
@@
     (stroke (width 0) (type default) (color 0 0 0 0))
   )
-  (wire (pts (xy 120.65 25.4) (xy 120.65 22.86))
+  (wire (pts (xy 120.65 22.86) (xy 120.65 24.384))
     (stroke (width 0) (type default) (color 0 0 0 0))
   )
@@
     (stroke (width 0) (type default) (color 0 0 0 0))
   )
+  (wire (pts (xy 120.65 28.956) (xy 127.508 28.956))
+    (stroke (width 0) (type default) (color 0 0 0 0))
+  )
   (wire (pts (xy 39.37 128.27) (xy 48.26 128.27))
     (stroke (width 0) (type default) (color 0 0 0 0))
@@
     (property "Reference" "SW8" (id 0) (at 148.59 88.9 0))
     (property "Value" "1825027-5" (id 1) (at 148.59 91.44 0))
-    (property "Footprint" "" (id 2) (at 148.59 95.25 0)
+    (property "Footprint" "wavbrd:Z_Switch_Edge_Omron" (id 2) (at 148.59 95.25 0)
       (effects (font (size 1.27 1.27)) hide)
     )
@@
     (pin "1")
   )
+  (symbol (lib_id "Connector:Conn_01x02_Male") (at 132.588 25.4 0) (mirror y) (unit 1)
+    (in_bom yes) (on_board yes)
+    (property "Reference" "J9" (id 0) (at 129.032 29.21 0))
+    (property "Value" "Conn_01x02_Male" (id 1) (at 134.874 30.988 0))
+    (property "Footprint" "" (id 2) (at 132.588 25.4 0)
+      (effects (font (size 1.27 1.27)) hide)
+    )
+    (property "Datasheet" "~" (id 3) (at 132.588 25.4 0)
+      (effects (font (size 1.27 1.27)) hide)
+    )
+    (pin "1")
+    (pin "2")
+  )
   (symbol (lib_id "power:VCC") (at 249.047 22.098 0) (unit 1)
     (in_bom yes) (on_board yes)
@@
       (reference "J8") (unit 1) (value "Conn_01x02_Male") (footprint "wavbrd:PinHeader_1x02_P2.54mm_Vertical")
     )
+    (path "/1a7f6efa-ef60-433d-acc0-6f9a9126bc57"
+      (reference "J9") (unit 1) (value "Conn_01x02_Male") (footprint "wavbrd:rumble_pins")
+    )
     (path "/d2da7f57-ee9e-4fd2-ab66-6ced21a875ef"
